File: Kicad/Doro56.kicad_pcb (KiCad board)
At the start: 2 copper layers, 175.4 x 115.2 mm, 77 parts, among them J1 MJ-4PP-9, SW1 SW_Push_45deg, SW10 SW_Push_45deg, SW11 SW_Push_45deg, SW12 SW_Push_45deg, SW13 SW_Push_45deg, SW14 SW_Push_45deg, SW15 SW_Push_45deg, SW16 SW_Push_45deg, SW17 SW_Push_45deg, SW18 SW_Push_45deg, SW19 SW_Push_45deg, SW2 SW_Push_45deg, SW20 SW_Push_45deg, SW21 SW_Push_45deg, SW22 SW_Push_45deg, SW23 SW_Push_45deg, SW24 SW_Push_45deg, SW25 SW_Push_45deg, SW26 SW_Push_45deg, SW27 SW_Push_45deg, SW28 SW_Push_45deg, SW29 SW_Push_45deg, SW3 SW_Push_45deg, SW30 SW_Push_45deg, SW31 SW_Push_45deg, SW32 SW_Push_45deg, SW33 RotaryEncoder_Switch, SW34 SW_SPDT, SW4 SW_Push_45deg, SW5 SW_Push_45deg, SW6 SW_Push_45deg, SW7 SW_Push_45deg, SW8 SW_Push_45deg, SW9 SW_Push_45deg, U1 ProMicro

Commit message: v1.1
v1.1 - Minor Edit
Caps and Enter Footprints: Changed to a reversible footprint (previously used two single key footprints rotated).
JST PH Footprint: Adjusted and relocated for increased flexibility.
PCB Cutout: Modified to remove blank space between Control and Alt keys, allowing space for a 402030 battery without increasing the case height clearance.
Plate: Slightly increased the cutout size for the rotary encoder.
Parts:
- removed the SW14 at (74.5, 86.1)
- BT1: footprint GHN:JST_PH_reversible -> GHN:JST_PH_reversible_vert
- SW13: footprint GHN:MX 1.75 STP 1.25 -> GHN:MX Rev 1U
- moved G*** 87.2 mm to (67.0, 48.5), turned to 0 degrees
- moved BT1 4.45 mm to (199.7, 93.4)
- moved BT2 1.33 mm to (199.7, 85.4)
- moved D13 0.51 mm to (93.7, 89.6)
- moved D9 0.51 mm to (136.5, 72.8)
- moved D28 0.51 mm to (189.2, 139.7)
- moved S29 0.51 mm to (171.0, 133.6)
- moved SW29 0.51 mm to (171.0, 133.6)
- moved D3 0.51 mm to (139.4, 49.1)
- moved SW9 0.51 mm to (128.7, 67.9)
- moved U1 0.51 mm to (210.3, 67.6)
- moved SW28 0.51 mm to (135.6, 129.2)
- moved SW2 0.51 mm to (111.5, 42.9)
- moved SW25 0.51 mm to (180.4, 115.5)
- moved D14 0.51 mm to (114.1, 89.6)
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- renumbered D15 to D14, D16 to D15, D17 to D16, D18 to D17, D19 to D18, D20 to D19, D22 to D21, D23 to D22, D24 to D23, D25 to D24, D26 to D25, D27 to D26, D28 to D27, D30 to D28, D31 to D29, D14 to D32, S14 to S13, S30 to S29, S20 to SS19, SW15 to SW14, SW16 to SW15, SW17 to SW16, SW18 to SW17, SW19 to SW18, SW20 to SW19, SW21 to SW20, SW22 to SW21, SW23 to SW22, SW24 to SW23, SW25 to SW24, SW26 to SW25, SW27 to SW26, SW28 to SW27, SW29 to SW28, SW30 to SW29, SW31 to SW30, SW32 to SW31
Connections:
- net SW33B renamed SW32B
Routing:
- net R4: track 186.0 -> 222.7 mm
- net C0: track 273.4 -> 286.8 mm, vias 3 -> 4
- net Net-(D13-A): track 24.2 -> 30.6 mm, vias 0 -> 1
- net /PSW: track 65.3 -> 71.2 mm
- net GND: track 21.8 -> 17.0 mm
Other:
- outline, holes or cut-outs redrawn
- board text added: "doro56 v1.1 github.com/gehennaxxiv"

Commit message: 1.2
Parts:
- removed SS19: MX_stab, PCM_marbastlib-mx:STAB_MX_2.25u
- added S19: MX_stab, PCM_marbastlib-mx:STAB_MX_2.25u, F.Cu at (68.2, 115.1)
- BT1: footprint GHN:JST_PH_reversible_vert -> GHN:JST_PH_2P_Reversible
- moved BT1 12.6 mm to (192.8, 104.0)
- moved D18 11.4 mm to (185.9, 111.8)
- moved D6 11.4 mm to (191.1, 69.3)
- moved D10 11.4 mm to (151.1, 82.6)
- moved SW20 11.4 mm to (73.0, 115.1)
- moved SW8 11.4 mm to (103.0, 77.0)
- moved BT2 11.4 mm to (195.0, 95.7)
- moved D15 11.4 mm to (129.5, 102.0)
- moved D25 11.4 mm to (183.5, 130.8)
- moved RST1 11.4 mm to (195.3, 135.3)
- moved J1 11.4 mm to (216.8, 103.7)
- moved H3 11.4 mm to (49.3, 46.2)
- moved SW14 11.4 mm to (101.1, 96.1)
- moved SW27 11.4 mm to (133.2, 139.9)
- moved SW34 11.4 mm to (211.9, 58.6)
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Routing:
- net /PSW: track 71.2 -> 72.7 mm
- net C0: track 286.8 -> 287.6 mm
- net C1: track 263.6 -> 264.4 mm
- net C2: track 239.0 -> 239.7 mm
Other:
- board text added: "Blk"
- board text added: "Red"
- board text added: "doro56 v1.2 github.com/gehennaxxiv"
- board text removed: "doro56 v1.1 github.com/gehennaxxiv"
